Commit message: fix: add real Franka inertials to panda.urdf; Isaac Sim 6.0.1 compatibility fixes
panda.urdf previously had zero <inertial> tags on any link, so RNEA was
computing dynamics with Pinocchio's placeholder inertias instead of real
Franka Panda mass properties. This surfaced as physically implausible
tau_res residuals (tens of Nm on gravity-bearing joints J2-J4) when first
compared against Isaac Sim's independently-massed Franka asset. Added
official franka_description inertial values for all links; re-running
data generation confirms residuals drop to a plausible, uniform
single-digit-Nm range across payloads 0/1/3 kg.

Also fixes generate_isaac_dataset.py for Isaac Sim 6.0.1: omni.isaac.* ->
isaacsim.* namespace migration, cmeel/pinocchio import path, moved Franka
USD asset path, TORQUE_LIMITS numpy dtype, world.stop() API change, and
buildReducedModel() to match RNEA's 7-DoF arm model to the 9-DoF URDF
(locking the 2 fixed finger joints). Adds tracking-error and joint-drive-gain
diagnostics used to rule out other explanations before finding the URDF gap.

Co-Authored-By: Claude Sonnet 5 <noreply@anthropic.com>

File: pinocchio_baseline/panda.urdf (robot description, URDF)
Before this commit: robot panda, 14 links, 13 joints
Links:
- link panda_hand: mass None -> 0.73
- link panda_leftfinger: mass None -> 0.015
- link panda_link0: mass None -> 0.629769
- link panda_link1: mass None -> 4.970684
- link panda_link2: mass None -> 0.646926
- link panda_link3: mass None -> 3.228604
- link panda_link4: mass None -> 3.587895
- link panda_link5: mass None -> 1.225946
- link panda_link6: mass None -> 1.666555
- link panda_link7: mass None -> 7.35522e-01
- link panda_rightfinger: mass None -> 0.015
