Commit message: feat(stage4): give the gripper real physics in MuJoCo, validated open/close
The hand/fingers in panda_arm_mujoco.xml were welded dead mass (no joints,
actuators, or collision) added earlier only to fix a gravity-compensation
mismatch -- physically incapable of opening, closing, or contacting anything.
They now have real prismatic joints, visual + collision geometry (fingers and
the previously-missing palm), an equality constraint coupling the two
fingers, and a properly-damped position actuator (retuned live from an
initially underdamped kp=500/no-kv, which overshot the joint's own range on
every move, to kp=30/kv=3).

panda_finger_joint1/2 were added into the arm's existing single
<ros2_control> block rather than a separate hardware component, after
confirming via mujoco_system_interface.cpp source that a second
MujocoSystemInterface instance would spin up a second, disconnected physics
simulation. The old mock_components-only hand system is removed.

launch/mujoco_franka_moveit.launch.py now spawns panda_hand_controller
(GripperActionController), already fully defined upstream and already
expected by MoveIt2's own gripper config, just never spawned before.

Validated live: open and close both succeed cleanly via panda_hand_controller's
gripper_cmd action (reached_goal: true, stalled: false), fingers stop against
each other without crossing.

Co-Authored-By: Claude Sonnet 5 <noreply@anthropic.com>

File: ros2_ws/src/pinn_franka_controller/urdf/panda_mujoco.ros2_control.xacro (robot description, xacro)
@@ -1,5 +1,20 @@
 <?xml version="1.0"?>
 <!--
-Stage 2/3: MuJoCo ros2_control hardware block for the Franka Panda arm.
+Stage 2/3: MuJoCo ros2_control hardware block for the Franka Panda arm AND hand/fingers.
+2026-07-22: panda_finger_joint1/2 were added directly into this SAME <ros2_control>
+"system" block (sharing this one "PandaMujocoSystem" hardware component), rather
+than as a separate hand-specific ros2_control block the way
+moveit_resources_panda_moveit_config's own panda_hand.ros2_control.xacro is used
+elsewhere (previously instantiated separately here too, as "PandaHandMockSystem",
+mock_components-only). This is required, not a style choice:
+MujocoSystemInterface::on_init() does `simulation_ = std::make_unique<MujocoSimulation>()`
+per hardware-component instance (confirmed by reading mujoco_system_interface.cpp from
+github.com/ros-controls/mujoco_ros2_control directly) — a second <ros2_control> "system"
+block using the mujoco plugin, even pointed at the same mujoco_model file, would spin up
+a SECOND, entirely disconnected physics simulation, with the hand's fingers floating in
+their own private void, mechanically detached from the arm they're physically bolted to
+in reality. Since the hand/fingers are already part of the same body tree in
+panda_arm_mujoco.xml as the arm, they must be driven by the arm's own single
+MujocoSystemInterface instance to end up in the same physical world.
 Clone of moveit_resources_panda_moveit_config's panda.ros2_control.xacro (same
 macro name/params, so it's a drop-in swap in a top-level xacro), adding a
@@ -48,5 +63,5 @@
             pids_config_file. In this mode MoveIt2's default position-mode
             panda_arm_controller CANNOT run (no position command interface for it
-            to claim) -- use this only when Milestone 1's path isn't needed.
+            to claim) — use this only when Milestone 1's path isn't needed.
         2026-07-21/22 correction: an earlier version of this comment claimed that
         in 'both' mode mujoco_ros2_control permanently locks each motor actuator
@@ -54,5 +69,5 @@
         effort commands (logged as a fixed per-joint "position control enabled
         (velocity, effort disabled)" state immune to controller-manager switching)
-        -- and blamed this for a session where Stage 3 effort commands produced
+        — and blamed this for a session where Stage 3 effort commands produced
         substantial, correctly time-varying torque but the arm stayed bit-for-bit
         frozen in position. That claim was written before the diagnostic it
@@ -63,5 +78,5 @@
         switches each joint from "position control enabled" to "effort control
         enabled" at runtime on controller switch, in 'both' mode, exactly as its
-        source implements -- confirmed by both the live log (a single switch
+        source implements — confirmed by both the live log (a single switch
         event, followed by "effort control enabled" persisting unchanged across a
         reset_world call and a full unload of panda_arm_controller, for the entire
@@ -115,4 +130,30 @@
             <xacro:panda_arm_joint joint_name="panda_joint6"/>
             <xacro:panda_arm_joint joint_name="panda_joint7"/>
+            <!-- Gripper: added 2026-07-22, see this file's header comment for why these
+                 live in this same <ros2_control> block instead of a separate one. Mirrors
+                 moveit_resources_panda_moveit_config's own panda_hand.ros2_control.xacro
+                 (command_interface only on finger_joint1, state-only on finger_joint2 —
+                 finger_joint2 is a physically-coupled follower via the MJCF's <equality>
+                 constraint, not independently commanded), except initial_value is 0.04
+                 (fully open) here rather than upstream's hardcoded 0.0 (closed): a safer
+                 default starting state for an eventual grasp demo, matching the MJCF
+                 "home" keyframe and MockGripperController's own default-open assumption. -->
+            <joint name="panda_finger_joint1">
+                <command_interface name="position"/>
+                <state_interface name="position">
+                  <param name="initial_value">0.04</param>
+                </state_interface>
+                <state_interface name="velocity">
+                    <param name="initial_value">0.0</param>
+                </state_interface>
+            </joint>
+            <joint name="panda_finger_joint2">
+                <state_interface name="position">
+                  <param name="initial_value">0.04</param>
+                </state_interface>
+                <state_interface name="velocity">
+                    <param name="initial_value">0.0</param>
+                </state_interface>
+            </joint>
         </ros2_control>
     </xacro:macro>

File: ros2_ws/src/pinn_franka_controller/urdf/panda_mujoco.urdf.xacro (robot description, xacro)
@@ -5,14 +5,15 @@
 (same shape: base panda.urdf unchanged, only the ros2_control include/instantiation
 swapped out).
-The hand IS instantiated as a ros2_control system (unlike panda_isaac.urdf.xacro,
-which dropped it for an Isaac-specific mimic-joint bug), but hardcoded to
-mock_components regardless of the arm's ros2_control_hardware_type arg: Stage 2/3
-only ever drives the 7 arm joints (pinn_controller_node's _JOINT_NAMES), so the
-gripper doesn't need real MuJoCo physics, but it DOES need a state_interface for
-panda_finger_joint1/2, or planning_scene_monitor never considers the robot's state
-"complete" (missing panda_finger_joint1) and MoveIt2's RViz plugin never renders
-anything at all, even though the arm joints are tracked fine. mock_components
-trivially mirrors commanded position back as state, exactly what's needed for a
-part of the robot this migration doesn't otherwise touch.
+2026-07-22: the hand/fingers are no longer a separate mock_components ros2_control
+system here. They previously were (hardcoded mock_components, "PandaHandMockSystem"),
+justified at the time by Stage 2/3 only ever driving the 7 arm joints — but mock
+joints are entirely synthetic (commanded position trivially mirrored back as state,
+zero physical presence), which became a real blocker once Stage 4 needed a gripper
+that can actually open/close/contact an object in the same physics world as the arm.
+panda_finger_joint1/2 are now declared inside panda_mujoco.ros2_control.xacro's own
+single <ros2_control> block instead (see that file's header comment for why: a
+second mujoco-plugin hardware component would spin up a second, disconnected
+simulation). The upstream panda_hand.ros2_control.xacro include below this comment
+is therefore no longer used.
 initial_positions_file is unchanged from moveit_resources_panda_moveit_config's own
 config/initial_positions.yaml (arm-only content, simulator-agnostic).
@@ -33,9 +34,6 @@
     <!-- Import our patched panda urdf file (real inertials added, see file header) -->
     <xacro:include filename="$(find pinn_franka_controller)/urdf/panda_mujoco_description.urdf" />
-    <!-- Import our MuJoCo ros2_control description (arm) -->
+    <!-- Import our MuJoCo ros2_control description (arm AND hand/fingers, see file header) -->
     <xacro:include filename="$(find pinn_franka_controller)/urdf/panda_mujoco.ros2_control.xacro" />
-    <!-- Hand: mock_components always, see file header -->
-    <xacro:include filename="$(find moveit_resources_panda_moveit_config)/config/panda_hand.ros2_control.xacro" />
     <xacro:panda_ros2_control name="PandaMujocoSystem" initial_positions_file="$(arg initial_positions_file)" ros2_control_hardware_type="$(arg ros2_control_hardware_type)" arm_control_mode="$(arg arm_control_mode)"/>
-    <xacro:panda_hand_ros2_control name="PandaHandMockSystem" ros2_control_hardware_type="mock_components"/>
 </robot>
