Commit message: fix(stage4): narrow panda_joint4/6/7 freeze from physics to ROS2/plugin layer
Multi-session Stage 4 grasping work (2026-07-20 through 2026-07-28), never
previously committed on this branch. Covers gripper physics, scene/object
setup, ArmMotionClient, and GraspExecutor (validated live across several
sessions), plus this session's deep-dive into the panda_joint4/6/7 freeze
that has blocked a working pick().

Key result this session: built a standalone diagnostic (stage4/debug_mujoco_internals.py)
that drives the project's own MJCF directly via the raw mujoco Python API,
bypassing ROS2 and the mujoco_ros2_control plugin entirely. Under the exact
torque that produces zero motion through the live ROS2 pipeline, joint4
moves completely freely. This rules out MuJoCo physics, the model file, and
joint4/6/7's physical parameters as the cause -- also rules out motion
planning (a fixed, deterministic bypass target froze identically to
MoveIt2's own varying solutions) and the trained PINN residual model
(RNEA+PD alone, via a new opt-in disable_residual flag on
ComputedTorquePDController, freezes identically). The bug is confirmed to
live in the mujoco_ros2_control plugin or the ros2_control command pathway
feeding it -- not yet root-caused at the C++ level.

Also fixes one real, previously-dismissed discrepancy: a project-local
ros2_ws/src/pinn_franka_controller/config/initial_positions.yaml now matches
the MJCF's own home keyframe exactly (the system-installed default disagreed
on joint2/4/7, joint7 by a full sign flip), wired in via
mujoco_franka_moveit.launch.py. NOT YET LIVE-VALIDATED -- the one test
attempt was invalidated by a sim-restart ordering mistake; re-testing this
correctly is the first thing to do next session, per SESSION.md.

New diagnostic tooling kept for reuse: stage4/test_direct_joint_bypass.py
(deterministic joint-space bypass of MoveIt2/OMPL), stage4/debug_mujoco_internals.py
(standalone MuJoCo internals inspector), ros2_ws/test_joint{4,6,7}_raw_torque.sh
(isolated single-joint torque tests), ros2_ws/launch_pinn_controller_no_residual.sh.

See SESSION.md and tracking/PROJECT_STATE.md for the full investigation
trail and next-session plan. No pick() is working yet; this commit captures
mid-debug state at the user's explicit request, an exception to the
project's normal not-mid-debug commit policy.

Co-Authored-By: Claude Sonnet 5 <noreply@anthropic.com>

File: ros2_ws/src/pinn_franka_controller/urdf/panda_mujoco_description.urdf (robot description, URDF)
Before this commit: robot panda, 12 links, 11 joints
Joints:
- joint panda_joint1: limit lower=-2.9671 upper=2.9671 effort=87 velocity=2.3925 -> lower=-2.8973 upper=2.8973 effort=87 velocity=2.1750
- joint panda_joint2: limit lower=-1.8326 upper=1.8326 effort=87 velocity=2.3925 -> lower=-1.7628 upper=1.7628 effort=87 velocity=2.1750
- joint panda_joint3: limit lower=-2.9671 upper=2.9671 effort=87 velocity=2.3925 -> lower=-2.8973 upper=2.8973 effort=87 velocity=2.1750
- joint panda_joint4: limit lower=-3.1416 upper=0.0873 effort=87 velocity=2.3925 -> lower=-3.0718 upper=-0.0698 effort=87 velocity=2.1750
- joint panda_joint5: limit lower=-2.9671 upper=2.9671 effort=12 velocity=2.8710 -> lower=-2.8973 upper=2.8973 effort=12 velocity=2.6100
- joint panda_joint6: limit lower=-0.0873 upper=3.8223 effort=12 velocity=2.8710 -> lower=-0.0175 upper=3.7525 effort=12 velocity=2.6100
- joint panda_joint7: limit lower=-2.9671 upper=2.9671 effort=12 velocity=2.8710 -> lower=-2.8973 upper=2.8973 effort=12 velocity=2.6100
